File: ScartPCB.kicad_pcb (KiCad board)
At the start: 4 copper layers, 39.5 x 21 mm, 55 parts, among them J1 Conn_02x10_Odd_Even, Q1 BC847W, Q2 BC857W, U1 TPS61040DBVR

Commit message: Add files via upload
Parts:
- CC1, CC2: value DNC -> 100uF
- CC3: value 50nF -> 22uF
Changed lines of the file:
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@@
     (property "Sheetfile" "ScartPCB.kicad_sch")
     (property "Sheetname" "")
-    (property "exclude_from_bom" "")
-    (attr smd exclude_from_bom)
+    (attr smd)
     (fp_text reference "CC2" (at 0.0254 -1.4986) (layer "F.SilkS")
       (effects (font (size 0.5 0.5) (thickness 0.1)))
     )
-    (fp_text value "DNC" (at 0 1.85) (layer "F.Fab") hide
+    (fp_text value "100uF" (at 0 1.85) (layer "F.Fab") hide
       (effects (font (size 1 1) (thickness 0.15)))
     )
@@
     (property "Sheetfile" "ScartPCB.kicad_sch")
     (property "Sheetname" "")
-    (property "exclude_from_bom" "")
-    (attr smd exclude_from_bom)
+    (attr smd)
     (fp_text reference "CC1" (at 0.1524 -1.524) (layer "F.SilkS")
       (effects (font (size 0.5 0.5) (thickness 0.1)))
     )
-    (fp_text value "DNC" (at 0 1.85) (layer "F.Fab") hide
+    (fp_text value "100uF" (at 0 1.85) (layer "F.Fab") hide
       (effects (font (size 1 1) (thickness 0.15)))
     )
@@
     (descr "Capacitor SMD 0603 (1608 Metric), square (rectangular) end terminal, IPC_7351 nominal, (Body size source: IPC-SM-782 page 76, https://www.pcb-3d.com/wordpress/wp-content/uploads/ipc-sm-782a_amendment_1_and_2.pdf), generated with kicad-footprint-generator")
     (tags "capacitor")
-    (property "Description" "50V 47nF X7R ±10% 0603 Multilayer Ceramic Capacitors MLCC - SMD/SMT ROHS ")
-    (property "Manufacturer" "Yaego")
-    (property "Manufacturer_Part_Number" "CC0603KRX7R9BB473")
+    (property "Description" " 10V 22uF X5R ±20% 0603 Multilayer Ceramic Capacitors MLCC - SMD/SMT ROHS ")
+    (property "Manufacturer" "Samsung")
+    (property "Manufacturer_Part_Number" "CL10A226MP8NUNE")
     (property "Package" "0603")
     (property "Sheetfile" "ScartPCB.kicad_sch")
@@
       (effects (font (size 0.5 0.5) (thickness 0.1)) (justify mirror))
     )
-    (fp_text value "50nF" (at 0 -1.43) (layer "B.Fab") hide
-      (effects (font (size 1 1) (thickness 0.15)) (justify mirror))
-    )
+    (fp_text value "22uF" (at 0 -1.43) (layer "B.Fab") hide
+      (effects (font (size 1 1) (thickness 0.15)) (justify mirror))
+    )
