File: ScartPCB.kicad_sch (KiCad schematic)
At the start: 55 parts, among them J1 Conn_02x10_Odd_Even, Q1 BC847W, Q2 BC857W, U1 TPS61040DBVR

Commit message: Add files via upload
Parts:
- CC1, CC2: value DNC -> 100uF; now in the parts list
- CC3: value 50nF -> 22uF; Manufacturer Yaego -> Samsung; Manufacturer_Part_Number CC0603KRX7R9BB473 -> CL10A226MP8NUNE
Other:
- moved on the sheet: CC1, CC3
Changed lines of the file:
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@@
     (stroke (width 0) (type dot) (color 0 0 0 0))
   )
-  (wire (pts (xy 140.97 59.69) (xy 162.56 59.69))
-    (stroke (width 0) (type default) (color 0 0 0 0))
-  )
   (wire (pts (xy 223.52 71.12) (xy 223.52 73.66))
     (stroke (width 0) (type default) (color 0 0 0 0))
@@
     (stroke (width 0) (type default) (color 0 0 0 0))
   )
-  (wire (pts (xy 140.97 63.5) (xy 151.13 63.5))
+  (wire (pts (xy 140.97 63.5) (xy 152.4 63.5))
     (stroke (width 0) (type default) (color 0 0 0 0))
   )
@@
     (stroke (width 0) (type default) (color 0 0 0 0))
   )
-  (wire (pts (xy 130.81 63.5) (xy 140.97 63.5))
+  (wire (pts (xy 129.54 63.5) (xy 140.97 63.5))
     (stroke (width 0) (type default) (color 0 0 0 0))
   )
@@
     (stroke (width 0) (type default) (color 0 0 0 0))
   )
-  (wire (pts (xy 151.13 63.5) (xy 151.13 66.04))
+  (wire (pts (xy 152.4 63.5) (xy 152.4 66.04))
     (stroke (width 0) (type default) (color 0 0 0 0))
   )
@@
     (stroke (width 0) (type default) (color 0 0 0 0))
   )
-  (wire (pts (xy 130.81 73.66) (xy 130.81 76.2))
+  (wire (pts (xy 129.54 73.66) (xy 129.54 76.2))
     (stroke (width 0) (type default) (color 0 0 0 0))
   )
@@
     (stroke (width 0) (type default) (color 0 0 0 0))
   )
-  (wire (pts (xy 130.81 66.04) (xy 130.81 63.5))
+  (wire (pts (xy 129.54 66.04) (xy 129.54 63.5))
     (stroke (width 0) (type default) (color 0 0 0 0))
   )
@@
     (stroke (width 0) (type default) (color 0 0 0 0))
   )
-  (wire (pts (xy 130.81 76.2) (xy 140.97 76.2))
+  (wire (pts (xy 129.54 76.2) (xy 140.97 76.2))
     (stroke (width 0) (type default) (color 0 0 0 0))
   )
@@
   )
   (wire (pts (xy 46.99 38.1) (xy 66.04 38.1))
+    (stroke (width 0) (type default) (color 0 0 0 0))
+  )
+  (wire (pts (xy 140.97 59.69) (xy 162.56 59.69))
     (stroke (width 0) (type default) (color 0 0 0 0))
   )
@@
     (stroke (width 0) (type default) (color 0 0 0 0))
   )
-  (wire (pts (xy 140.97 76.2) (xy 151.13 76.2))
+  (wire (pts (xy 140.97 76.2) (xy 152.4 76.2))
     (stroke (width 0) (type default) (color 0 0 0 0))
   )
@@
     (stroke (width 0) (type default) (color 0 0 0 0))
   )
-  (wire (pts (xy 151.13 76.2) (xy 151.13 73.66))
+  (wire (pts (xy 152.4 76.2) (xy 152.4 73.66))
     (stroke (width 0) (type default) (color 0 0 0 0))
   )
@@
     (pin "1")
   )
-  (symbol (lib_id "Device:C") (at 130.81 69.85 0) (mirror x) (unit 1)
-    (in_bom no) (on_board yes)
-    (property "Reference" "CC1" (id 0) (at 133.35 71.12 0)
-      (effects (font (size 1.27 1.27)) (justify left))
-    )
-    (property "Value" "DNC" (id 1) (at 133.35 68.5799 0)
-      (effects (font (size 1.27 1.27)) (justify left))
-    )
-    (property "Footprint" "Capacitor_SMD:C_1206_3216Metric" (id 2) (at 131.7752 66.04 0)
-      (effects (font (size 1.27 1.27)) hide)
-    )
-    (property "Datasheet" "https://eu.mouser.com/datasheet/2/281/1/GRM31CR61A107ME05_01A-2066674.pdf" (id 3) (at 130.81 69.85 0)
-      (effects (font (size 1.27 1.27)) hide)
-    )
-    (property "Manufacturer" "Murata Electronics" (id 4) (at 130.81 69.85 0)
-      (effects (font (size 1.27 1.27)) hide)
-    )
-    (property "Manufacturer_Part_Number" "GRM31CR61A107ME05L" (id 5) (at 130.81 69.85 0)
-      (effects (font (size 1.27 1.27)) hide)
-    )
-    (property "Description" " 10V 100uF X5R ±20% 1206 Multilayer Ceramic Capacitors MLCC - SMD/SMT ROHS " (id 6) (at 130.81 69.85 0)
-      (effects (font (size 1.27 1.27)) hide)
-    )
-    (property "Package" "1206" (id 7) (at 130.81 69.85 0)
+  (symbol (lib_id "Device:C") (at 129.54 69.85 0) (mirror x) (unit 1)
+    (in_bom yes) (on_board yes)
+    (property "Reference" "CC1" (id 0) (at 132.08 68.58 0)
+      (effects (font (size 1.27 1.27)) (justify left))
+    )
+    (property "Value" "100uF" (id 1) (at 132.08 71.12 0)
+      (effects (font (size 1.27 1.27)) (justify left))
+    )
+    (property "Footprint" "Capacitor_SMD:C_1206_3216Metric" (id 2) (at 130.5052 66.04 0)
+      (effects (font (size 1.27 1.27)) hide)
+    )
+    (property "Datasheet" "https://eu.mouser.com/datasheet/2/281/1/GRM31CR61A107ME05_01A-2066674.pdf" (id 3) (at 129.54 69.85 0)
+      (effects (font (size 1.27 1.27)) hide)
+    )
+    (property "Manufacturer" "Murata Electronics" (id 4) (at 129.54 69.85 0)
+      (effects (font (size 1.27 1.27)) hide)
+    )
+    (property "Manufacturer_Part_Number" "GRM31CR61A107ME05L" (id 5) (at 129.54 69.85 0)
+      (effects (font (size 1.27 1.27)) hide)
+    )
+    (property "Description" " 10V 100uF X5R ±20% 1206 Multilayer Ceramic Capacitors MLCC - SMD/SMT ROHS " (id 6) (at 129.54 69.85 0)
+      (effects (font (size 1.27 1.27)) hide)
+    )
+    (property "Package" "1206" (id 7) (at 129.54 69.85 0)
       (effects (font (size 1.27 1.27)) hide)
     )
@@
     (pin "1")
   )
-  (symbol (lib_id "Device:C") (at 151.13 69.85 0) (mirror x) (unit 1)
-    (in_bom yes) (on_board yes)
-    (property "Reference" "CC3" (id 0) (at 153.67 71.12 0)
-      (effects (font (size 1.27 1.27)) (justify left))
-    )
-    (property "Value" "50nF" (id 1) (at 153.67 68.58 0)
-      (effects (font (size 1.27 1.27)) (justify left))
-    )
-    (property "Footprint" "Capacitor_SMD:C_0603_1608Metric" (id 2) (at 152.0952 66.04 0)
-      (effects (font (size 1.27 1.27)) hide)
-    )
-    (property "Datasheet" "https://www.mouser.it/datasheet/2/447/UPY_NP0X5R_01005_4V_to_25V_V10-3003057.pdf" (id 3) (at 151.13 69.85 0)
-      (effects (font (size 1.27 1.27)) hide)
-    )
-    (property "Manufacturer" "Yaego" (id 4) (at 151.13 69.85 0)
-      (effects (font (size 1.27 1.27)) hide)
-    )
-    (property "Manufacturer_Part_Number" "CC0603KRX7R9BB473" (id 5) (at 151.13 69.85 0)
-      (effects (font (size 1.27 1.27)) hide)
-    )
-    (property "Description" "50V 47nF X7R ±10% 0603 Multilayer Ceramic Capacitors MLCC - SMD/SMT ROHS " (id 6) (at 151.13 69.85 0)
-      (effects (font (size 1.27 1.27)) hide)
-    )
-    (property "Package" "0603" (id 7) (at 151.13 69.85 0)
+  (symbol (lib_id "Device:C") (at 152.4 69.85 0) (mirror x) (unit 1)
+    (in_bom yes) (on_board yes)
+    (property "Reference" "CC3" (id 0) (at 154.94 68.58 0)
+      (effects (font (size 1.27 1.27)) (justify left))
+    )
+    (property "Value" "22uF" (id 1) (at 154.94 71.12 0)
+      (effects (font (size 1.27 1.27)) (justify left))
+    )
+    (property "Footprint" "Capacitor_SMD:C_0603_1608Metric" (id 2) (at 153.3652 66.04 0)
+      (effects (font (size 1.27 1.27)) hide)
+    )
+    (property "Datasheet" "https://eu.mouser.com/datasheet/2/585/MLCC-1837944.pdf" (id 3) (at 152.4 69.85 0)
+      (effects (font (size 1.27 1.27)) hide)
+    )
+    (property "Manufacturer" "Samsung" (id 4) (at 152.4 69.85 0)
+      (effects (font (size 1.27 1.27)) hide)
+    )
+    (property "Manufacturer_Part_Number" "CL10A226MP8NUNE" (id 5) (at 152.4 69.85 0)
+      (effects (font (size 1.27 1.27)) hide)
+    )
+    (property "Description" " 10V 22uF X5R ±20% 0603 Multilayer Ceramic Capacitors MLCC - SMD/SMT ROHS " (id 6) (at 152.4 69.85 0)
+      (effects (font (size 1.27 1.27)) hide)
+    )
+    (property "Package" "0603" (id 7) (at 152.4 69.85 0)
       (effects (font (size 1.27 1.27)) hide)
     )
@@
   )
   (symbol (lib_id "Device:C") (at 140.97 69.85 0) (mirror x) (unit 1)
-    (in_bom no) (on_board yes)
-    (property "Reference" "CC2" (id 0) (at 143.51 71.12 0)
-      (effects (font (size 1.27 1.27)) (justify left))
-    )
-    (property "Value" "DNC" (id 1) (at 143.51 68.5799 0)
+    (in_bom yes) (on_board yes)
+    (property "Reference" "CC2" (id 0) (at 143.51 68.58 0)
+      (effects (font (size 1.27 1.27)) (justify left))
+    )
+    (property "Value" "100uF" (id 1) (at 143.51 71.12 0)
       (effects (font (size 1.27 1.27)) (justify left))
     )
@@
     )
     (path "/61392744-303e-4387-bfcf-9016066fe6f6"
-      (reference "CC1") (unit 1) (value "DNC") (footprint "Capacitor_SMD:C_1206_3216Metric")
+      (reference "CC1") (unit 1) (value "100uF") (footprint "Capacitor_SMD:C_1206_3216Metric")
     )
     (path "/794b2b0a-195b-44a9-81a7-664c10a9f700"
-      (reference "CC2") (unit 1) (value "DNC") (footprint "Capacitor_SMD:C_1206_3216Metric")
+      (reference "CC2") (unit 1) (value "100uF") (footprint "Capacitor_SMD:C_1206_3216Metric")
     )
     (path "/66c4f955-5301-4c69-a922-8aa05852692f"
-      (reference "CC3") (unit 1) (value "50nF") (footprint "Capacitor_SMD:C_0603_1608Metric")
+      (reference "CC3") (unit 1) (value "22uF") (footprint "Capacitor_SMD:C_0603_1608Metric")
     )
     (path "/eacc3101-923b-4cf6-83db-d6363a7f5e73"
